File: PiroSensor_Rev1/PiroSensor_Rev1.kicad_pcb (KiCad board)
At the start: 2 copper layers, 42 x 60 mm, 39 parts, among them IC2 EFR32FG23L020F128GM40-C, IC3 PYD1398, J1 MY-18650-01, J2 MY-18650-01, Q1 AO3401A, SW1 SW_SPDT, SW2 SW_Push, U1 LM358

Commit message: feat: atualização do projeto - 2026-06-05 15:12
Parts:
- added C13: C, Capacitor_SMD:C_0603_1608Metric, F.Cu at (145.8, 68.4)
- added C14: 7,2pF, Capacitor_SMD:C_0603_1608Metric, F.Cu at (145.8, 71.4)
- added C15: C, Capacitor_SMD:C_0603_1608Metric, F.Cu at (138.2, 74.6)
- added C16: 220pF, Capacitor_SMD:C_0603_1608Metric, F.Cu at (143.5, 75.2)
- added C17: 1,9pF, Capacitor_SMD:C_0603_1608Metric, F.Cu at (142.0, 66.1)
- added C18: 1,3pF, Capacitor_SMD:C_0603_1608Metric, F.Cu at (145.7, 74.4)
- added C19: 1uF, Capacitor_SMD:C_0603_1608Metric, F.Cu at (137.9, 60.9)
- added C20: 100pF, Capacitor_SMD:C_0603_1608Metric, F.Cu at (137.9, 62.5)
- added C21: 470nF, Capacitor_SMD:C_0603_1608Metric, F.Cu at (147.6, 62.4)
- added C22: 100pF, Capacitor_SMD:C_0603_1608Metric, F.Cu at (147.6, 63.9)
- added C23: 1,5pF, Capacitor_SMD:C_0603_1608Metric, F.Cu at (147.6, 59.3)
- added C24: 1,5pF, Capacitor_SMD:C_0603_1608Metric, F.Cu at (147.6, 57.8)
- added C25: 10uF, Capacitor_SMD:C_0603_1608Metric, F.Cu at (144.5, 53.1)
- added C26: 100nF, Capacitor_SMD:C_0603_1608Metric, F.Cu at (144.5, 54.6)
- added C27: 10nF, Capacitor_SMD:C_0603_1608Metric, F.Cu at (141.4, 54.6)
- added C28: 1uF, Capacitor_SMD:C_0603_1608Metric, F.Cu at (141.4, 53.1)
- added C29: 100nF, Capacitor_SMD:C_0603_1608Metric, F.Cu at (141.4, 51.6)
- added C30: 1uF, Capacitor_SMD:C_0603_1608Metric, F.Cu at (141.4, 50.1)
- added C31: 100nF, Capacitor_SMD:C_0603_1608Metric, F.Cu at (147.6, 53.1)
- added C32: 1uF, Capacitor_SMD:C_0603_1608Metric, F.Cu at (147.6, 51.6)
- added C33: 100nF, Capacitor_SMD:C_0603_1608Metric, F.Cu at (144.5, 50.1)
- added C34: 4,7uF, Capacitor_SMD:C_0603_1608Metric, F.Cu at (147.6, 54.6)
- added FB1: FerriteBead, Inductor_SMD:L_0603_1608Metric, F.Cu at (137.9, 59.3)
- added FB2: FerriteBead, Inductor_SMD:L_0603_1608Metric, F.Cu at (147.6, 60.9)
- added FB3: FerriteBead, Inductor_SMD:L_0603_1608Metric, F.Cu at (147.6, 65.4)
- added L1: 1,5nH, Inductor_SMD:L_0603_1608Metric, F.Cu at (143.5, 66.1)
- added L2: 1,3nH, Inductor_SMD:L_0603_1608Metric, F.Cu at (143.5, 69.1)
- added L3: 13nH, Inductor_SMD:L_0603_1608Metric, F.Cu at (143.5, 72.1)
- added L4: 18nH, Inductor_SMD:L_0603_1608Metric, F.Cu at (140.5, 75.3)
- added L5: 2,2uH, Inductor_SMD:L_0603_1608Metric, F.Cu at (147.6, 56.2)
- added Y1: 39MHz, SamacSys_Parts:ABM8AIG25000MHZ122ZT3, F.Cu at (138.9, 69.7)
- D1, D2: footprint Diode_SMD:D_MiniMELF -> Diode_SMD:D_SOD-323
- SW2: footprint Button_Switch_SMD:SW_Push_1P1T_NO_CK_KSC6xxG -> Button_Switch_SMD:SW_Push_1P1T_NO_E-Switch_TL3301NxxxxxG
- moved R14 31.4 mm to (127.0, 58.8), turned to 90 degrees
- moved C1 31.2 mm to (124.6, 68.0), turned to -90 degrees
- moved C3 29.4 mm to (123.0, 71.1), turned to -90 degrees
- moved C2 29.4 mm to (123.0, 68.0), turned to 90 degrees
- moved R1 29.2 mm to (124.6, 64.9), turned to -90 degrees
- moved C4 27.8 mm to (121.5, 71.1), turned to -90 degrees
- moved R3 27.5 mm to (128.6, 71.9), turned to 180 degrees
- moved C6 26.7 mm to (119.9, 71.1), turned to -90 degrees
- moved C10 26.5 mm to (121.7, 60.0), turned to 180 degrees
- moved R2 25.6 mm to (126.2, 71.1), turned to -90 degrees
- moved C5 23.4 mm to (117.0, 71.1), turned to -90 degrees
- moved R4 23.0 mm to (124.6, 71.1), turned to -90 degrees
- moved C9 22.7 mm to (118.7, 60.0)
- moved R11 21.4 mm to (121.7, 57.0)
- moved D2 21.1 mm to (114.8, 75.5)
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Connections:
- ANT1 pad 1: unconnected-(ANT1-FEED-Pad1) -> Net-(ANT1-FEED)
- IC2 pad 10: unconnected-(IC2-HFXTAL_O-Pad10) -> Net-(IC2-HFXTAL_O)
- IC2 pad 12: unconnected-(IC2-RFVDD-Pad12) -> Net-(IC2-RFVDD)
- IC2 pad 13: unconnected-(IC2-RFVSS-Pad13) -> GND
- IC2 pad 14: unconnected-(IC2-SUBG_I1-Pad14) -> Net-(IC2-SUBG_I1)
- IC2 pad 15: unconnected-(IC2-SUBG_I0-Pad15) -> Net-(IC2-SUBG_I0)
- IC2 pad 16: unconnected-(IC2-SUBG_O1-Pad16) -> Net-(IC2-SUBG_O1)
- IC2 pad 17: unconnected-(IC2-SUBG_O0-Pad17) -> Net-(IC2-SUBG_O0)
- IC2 pad 18: unconnected-(IC2-PAVDD-Pad18) -> Net-(IC2-PAVDD)
- IC2 pad 30: unconnected-(IC2-DECOUPLE-Pad30) -> Net-(IC2-DECOUPLE)
- IC2 pad 31: unconnected-(IC2-VREGSW-Pad31) -> Net-(IC2-VREGSW)
- IC2 pad 32: unconnected-(IC2-VREGVDD-Pad32) -> +3V0
- IC2 pad 33: unconnected-(IC2-VREGVSS-Pad33) -> GND
- IC2 pad 34: unconnected-(IC2-DVDD-Pad34) -> +3V0
- IC2 pad 35: unconnected-(IC2-AVDD-Pad35) -> +3V0
- IC2 pad 36: unconnected-(IC2-IOVDD-Pad36) -> +3V0
- IC2 pad 41: unconnected-(IC2-EP-Pad41) -> GND
- IC2 pad 9: unconnected-(IC2-HFXTAL_I-Pad9) -> Net-(IC2-HFXTAL_I)
