File: PiroSensor_Rev1/amplificador.kicad_sch (KiCad schematic)
At the start: 30 parts, among them IC3 PYD1398, U1 LM358

Commit message: feat: atualização do projeto - 2026-06-05 15:12
Parts:
- D1, D2: footprint Diode_SMD:D_MiniMELF -> Diode_SMD:D_SOD-323
Changed lines of the file:
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@@
 			)
 		)
-		(property "Footprint" "Diode_SMD:D_MiniMELF"
+		(property "Footprint" "Diode_SMD:D_SOD-323"
 			(at 151.13 145.415 0)
 			(hide yes)
@@
 			)
 		)
-		(property "Footprint" "Diode_SMD:D_MiniMELF"
+		(property "Footprint" "Diode_SMD:D_SOD-323"
 			(at 151.13 146.685 0)
 			(hide yes)
